File: pcb/keyboard_pcb.kicad_sch (KiCad schematic)
At the start: 23 parts, among them J1 TRRS, K00 KEYSW, K01 KEYSW, K02 KEYSW, K03 KEYSW, K04 KEYSW, K05 KEYSW, K10 KEYSW, K11 KEYSW, K12 KEYSW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

Commit message: Mod to 36 keys and add silkscreen
Parts:
- removed K00, K10, K20: KEYSW, keyswitches:SW_PG1350_reversible, symbol keyboard_parts:KEYSW
Connections:
- net k01: no longer U1.37 (PB10)
- net k00: no longer names the net of U1.35 (PB1)
- net k20: no longer names the net of U1.29 (PA3)
- no-connect marks 13 -> 16
Changed lines of the file:
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@@
   (no_connect (at 91.44 34.29))
   (no_connect (at 50.8 77.47))
+  (no_connect (at 91.44 41.91))
+  (no_connect (at 91.44 46.99))
+  (no_connect (at 91.44 62.23))
   (wire (pts (xy 149.86 60.96) (xy 154.94 60.96))
     (stroke (width 0) (type default) (color 0 0 0 0))
@@
     (stroke (width 0) (type default) (color 0 0 0 0))
   )
-  (wire (pts (xy 124.46 45.72) (xy 129.54 45.72))
-    (stroke (width 0) (type default) (color 0 0 0 0))
-  )
   (wire (pts (xy 200.66 60.96) (xy 205.74 60.96))
     (stroke (width 0) (type default) (color 0 0 0 0))
@@
     (stroke (width 0) (type default) (color 0 0 0 0))
   )
-  (wire (pts (xy 91.44 41.91) (xy 97.79 41.91))
-    (stroke (width 0) (type default) (color 0 0 0 0))
-  )
   (wire (pts (xy 175.26 60.96) (xy 180.34 60.96))
     (stroke (width 0) (type default) (color 0 0 0 0))
@@
     (stroke (width 0) (type default) (color 0 0 0 0))
   )
-  (wire (pts (xy 144.78 63.5) (xy 144.78 60.96))
-    (stroke (width 0) (type default) (color 0 0 0 0))
-  )
   (wire (pts (xy 246.38 48.26) (xy 246.38 45.72))
     (stroke (width 0) (type default) (color 0 0 0 0))
@@
     (stroke (width 0) (type default) (color 0 0 0 0))
   )
-  (wire (pts (xy 144.78 48.26) (xy 144.78 45.72))
-    (stroke (width 0) (type default) (color 0 0 0 0))
-  )
-  (wire (pts (xy 91.44 62.23) (xy 97.79 62.23))
-    (stroke (width 0) (type default) (color 0 0 0 0))
-  )
   (wire (pts (xy 93.98 36.83) (xy 93.98 30.48))
     (stroke (width 0) (type default) (color 0 0 0 0))
@@
     (stroke (width 0) (type default) (color 0 0 0 0))
   )
-  (wire (pts (xy 124.46 60.96) (xy 129.54 60.96))
-    (stroke (width 0) (type default) (color 0 0 0 0))
-  )
-  (wire (pts (xy 144.78 33.02) (xy 144.78 30.48))
-    (stroke (width 0) (type default) (color 0 0 0 0))
-  )
   (wire (pts (xy 195.58 48.26) (xy 195.58 45.72))
     (stroke (width 0) (type default) (color 0 0 0 0))
@@
     (stroke (width 0) (type default) (color 0 0 0 0))
   )
-  (wire (pts (xy 124.46 30.48) (xy 129.54 30.48))
-    (stroke (width 0) (type default) (color 0 0 0 0))
-  )
   (wire (pts (xy 93.98 30.48) (xy 97.79 30.48))
     (stroke (width 0) (type default) (color 0 0 0 0))
@@
     (stroke (width 0) (type default) (color 0 0 0 0))
   )
-  (wire (pts (xy 91.44 46.99) (xy 97.79 46.99))
-    (stroke (width 0) (type default) (color 0 0 0 0))
-  )
   (wire (pts (xy 91.44 57.15) (xy 97.79 57.15))
     (stroke (width 0) (type default) (color 0 0 0 0))
@@
     (stroke (width 0) (type default) (color 0 0 0 0))
   )
-  (label "k20" (at 97.79 62.23 0)
-    (effects (font (size 1.27 1.27)) (justify left bottom))
-  )
   (label "TX" (at 64.77 120.65 0)
     (effects (font (size 1.27 1.27)) (justify left bottom))
   )
-  (label "k01" (at 97.79 41.91 0)
-    (effects (font (size 1.27 1.27)) (justify left bottom))
-  )
   (label "k03" (at 44.45 41.91 0)
     (effects (font (size 1.27 1.27)) (justify left bottom))
@@
     (effects (font (size 1.27 1.27)) (justify left bottom))
   )
-  (label "k00" (at 124.46 30.48 0)
-    (effects (font (size 1.27 1.27)) (justify left bottom))
-  )
   (label "k10" (at 44.45 74.93 0)
     (effects (font (size 1.27 1.27)) (justify left bottom))
@@
     (effects (font (size 1.27 1.27)) (justify left bottom))
   )
-  (label "k10" (at 124.46 45.72 0)
-    (effects (font (size 1.27 1.27)) (justify left bottom))
-  )
-  (label "k00" (at 97.79 46.99 0)
-    (effects (font (size 1.27 1.27)) (justify left bottom))
-  )
   (label "k21" (at 97.79 59.69 0)
     (effects (font (size 1.27 1.27)) (justify left bottom))
@@
   )
   (label "k23" (at 97.79 54.61 0)
-    (effects (font (size 1.27 1.27)) (justify left bottom))
-  )
-  (label "k20" (at 124.46 60.96 0)
     (effects (font (size 1.27 1.27)) (justify left bottom))
   )
@@
     (pin "1")
   )
-  (symbol (lib_id "keyboard_parts:KEYSW") (at 137.16 30.48 0) (mirror y) (unit 1)
-    (in_bom yes) (on_board yes) (fields_autoplaced)
-    (property "Reference" "K00" (id 0) (at 137.16 24.13 0)
-      (effects (font (size 1.524 1.524)))
-    )
-    (property "Value" "KEYSW" (id 1) (at 137.16 33.02 0)
-      (effects (font (size 1.524 1.524)) hide)
-    )
-    (property "Footprint" "keyswitches:SW_PG1350_reversible" (id 2) (at 137.16 30.48 0)
-      (effects (font (size 1.524 1.524)) hide)
-    )
-    (property "Datasheet" "" (id 3) (at 137.16 30.48 0)
-      (effects (font (size 1.524 1.524)))
-    )
-    (pin "1")
-    (pin "2")
-  )
   (symbol (lib_id "keyboard_parts:KEYSW") (at 264.16 45.72 0) (mirror y) (unit 1)
     (in_bom yes) (on_board yes) (fields_autoplaced)
@@
     (pin "1")
     (pin "2")
-  )
-  (symbol (lib_id "power:GND") (at 144.78 48.26 0) (unit 1)
-    (in_bom yes) (on_board yes)
-    (property "Reference" "#PWR0107" (id 0) (at 144.78 54.61 0)
-      (effects (font (size 1.27 1.27)) hide)
-    )
-    (property "Value" "GND" (id 1) (at 144.78 53.34 0))
-    (property "Footprint" "" (id 2) (at 144.78 48.26 0)
-      (effects (font (size 1.27 1.27)) hide)
-    )
-    (property "Datasheet" "" (id 3) (at 144.78 48.26 0)
-      (effects (font (size 1.27 1.27)) hide)
-    )
-    (pin "1")
   )
   (symbol (lib_id "power:GND") (at 195.58 63.5 0) (unit 1)
@@
     (pin "4")
   )
-  (symbol (lib_id "keyboard_parts:KEYSW") (at 137.16 60.96 0) (mirror y) (unit 1)
-    (in_bom yes) (on_board yes)
-    (property "Reference" "K20" (id 0) (at 137.16 55.88 0)
-      (effects (font (size 1.524 1.524)))
-    )
-    (property "Value" "KEYSW" (id 1) (at 137.16 63.5 0)
-      (effects (font (size 1.524 1.524)) hide)
-    )
-    (property "Footprint" "keyswitches:SW_PG1350_reversible" (id 2) (at 137.16 60.96 0)
-      (effects (font (size 1.524 1.524)) hide)
-    )
-    (property "Datasheet" "" (id 3) (at 137.16 60.96 0)
-      (effects (font (size 1.524 1.524)))
-    )
-    (pin "1")
-    (pin "2")
-  )
   (symbol (lib_id "power:GND") (at 271.78 48.26 0) (unit 1)
     (in_bom yes) (on_board yes)
@@
     (pin "2")
   )
-  (symbol (lib_id "keyboard_parts:KEYSW") (at 137.16 45.72 0) (mirror y) (unit 1)
-    (in_bom yes) (on_board yes) (fields_autoplaced)
-    (property "Reference" "K10" (id 0) (at 137.16 39.37 0)
-      (effects (font (size 1.524 1.524)))
-    )
-    (property "Value" "KEYSW" (id 1) (at 137.16 48.26 0)
-      (effects (font (size 1.524 1.524)) hide)
-    )
-    (property "Footprint" "keyswitches:SW_PG1350_reversible" (id 2) (at 137.16 45.72 0)
-      (effects (font (size 1.524 1.524)) hide)
-    )
-    (property "Datasheet" "" (id 3) (at 137.16 45.72 0)
-      (effects (font (size 1.524 1.524)))
-    )
-    (pin "1")
-    (pin "2")
-  )
   (symbol (lib_id "keyboard_parts:KEYSW") (at 162.56 30.48 0) (mirror y) (unit 1)
     (in_bom yes) (on_board yes)
@@
     (pin "1")
   )
-  (symbol (lib_id "power:GND") (at 144.78 33.02 0) (unit 1)
-    (in_bom yes) (on_board yes)
-    (property "Reference" "#PWR0109" (id 0) (at 144.78 39.37 0)
-      (effects (font (size 1.27 1.27)) hide)
-    )
-    (property "Value" "GND" (id 1) (at 144.78 38.1 0))
-    (property "Footprint" "" (id 2) (at 144.78 33.02 0)
-      (effects (font (size 1.27 1.27)) hide)
-    )
-    (property "Datasheet" "" (id 3) (at 144.78 33.02 0)
-      (effects (font (size 1.27 1.27)) hide)
-    )
-    (pin "1")
-  )
   (symbol (lib_id "power:GND") (at 33.02 80.01 0) (unit 1)
     (in_bom yes) (on_board yes) (fields_autoplaced)
@@
     )
     (property "Datasheet" "" (id 3) (at 220.98 63.5 0)
-      (effects (font (size 1.27 1.27)) hide)
-    )
-    (pin "1")
-  )
-  (symbol (lib_id "power:GND") (at 144.78 63.5 0) (unit 1)
-    (in_bom yes) (on_board yes)
-    (property "Reference" "#PWR0108" (id 0) (at 144.78 69.85 0)
-      (effects (font (size 1.27 1.27)) hide)
-    )
-    (property "Value" "GND" (id 1) (at 144.78 68.58 0))
-    (property "Footprint" "" (id 2) (at 144.78 63.5 0)
-      (effects (font (size 1.27 1.27)) hide)
-    )
-    (property "Datasheet" "" (id 3) (at 144.78 63.5 0)
       (effects (font (size 1.27 1.27)) hide)
     )
@@
       (reference "#PWR0106") (unit 1) (value "GND") (footprint "")
     )
-    (path "/3e44ea14-8ee3-46fe-9ebd-10f5682c06c5"
-      (reference "#PWR0107") (unit 1) (value "GND") (footprint "")
-    )
-    (path "/f285bac1-bf5d-4300-80bd-ca1a79d56d03"
-      (reference "#PWR0108") (unit 1) (value "GND") (footprint "")
-    )
-    (path "/cf9971d6-27ee-4856-8e31-d3769822fc2a"
-      (reference "#PWR0109") (unit 1) (value "GND") (footprint "")
-    )
     (path "/f587ddb8-6759-41fb-857c-4c66d5d9f816"
       (reference "#PWR0110") (unit 1) (value "GND") (footprint "")
@@
       (reference "J1") (unit 1) (value "TRRS") (footprint "Keebio-Parts:TRRS-PJ-320A")
     )
-    (path "/2cd2ee6e-af2a-43ce-aa7e-58b5c17fc3c8"
-      (reference "K00") (unit 1) (value "KEYSW") (footprint "keyswitches:SW_PG1350_reversible")
-    )
     (path "/b5cead6f-dcdf-499e-bfad-67a021a50a6a"
       (reference "K01") (unit 1) (value "KEYSW") (footprint "keyswitches:SW_PG1350_reversible")
@@
       (reference "K05") (unit 1) (value "KEYSW") (footprint "keyswitches:SW_PG1350_reversible")
     )
-    (path "/b4241be9-1d03-4b7d-96ed-4ef26aa15e0b"
-      (reference "K10") (unit 1) (value "KEYSW") (footprint "keyswitches:SW_PG1350_reversible")
-    )
     (path "/5c3d7d74-dde3-4ed7-8c8b-9834e1dad91c"
       (reference "K11") (unit 1) (value "KEYSW") (footprint "keyswitches:SW_PG1350_reversible")
@@
       (reference "K15") (unit 1) (value "KEYSW") (footprint "keyswitches:SW_PG1350_reversible")
     )
-    (path "/9dd6772e-ed36-40d9-bc93-987b987d9bc6"
-      (reference "K20") (unit 1) (value "KEYSW") (footprint "keyswitches:SW_PG1350_reversible")
-    )
     (path "/e0e7955b-d8e1-40e6-8c21-1d8aac3d0cb0"
